Commit message: Added collisions to urdf

File: urdf/efim.urdf (robot description, URDF)
Before this commit: robot myfirst, 7 links, 6 joints
Links:
- link base_link: geometry collision cylinder length=1.04775 radius=0.2032; visual cylinder length=1.04775 radius=0.2032
- link base_lower_link: geometry collision box size=0.41148 0.30988 0.05588; visual box size=0.41148 0.30988 0.05588
- link hitch_front_link: geometry collision cylinder length=0.1524 radius=0.01; visual cylinder length=0.1524 radius=0.01
- link wheel_front_left: geometry collision cylinder length=0.1524 radius=0.01; visual cylinder length=0.0508 radius=0.0762
- link wheel_front_right: geometry collision cylinder length=0.1524 radius=0.01; visual cylinder length=0.0508 radius=0.0762
- link wheel_rear_left: geometry collision cylinder length=0.1524 radius=0.01; visual cylinder length=0.0508 radius=0.0762
- link wheel_rear_right: geometry collision cylinder length=0.1524 radius=0.01; visual cylinder length=0.0508 radius=0.0762
