Commit message: updates

File: urdf/sherpa.urdf.xacro (robot description, xacro)
@@ -156,5 +156,5 @@
     </sensor>
 </gazebo>
-<gazebo reference="camera_link">
+<gazebo reference="laser_link">
     <material>Gazebo/Blue</material>
     <sensor type="gpu_ray" name="hokuyo">
@@ -179,5 +179,5 @@
       <plugin name="gpu_laser" filename="libgazebo_ros_gpu_laser.so">
         <topicName>/scan</topicName>
-        <frameName>camera_link</frameName>
+        <frameName>laser_link</frameName>
       </plugin>
     </sensor>
@@ -189,5 +189,5 @@
     <origin rpy="0 0 0" xyz="0.2 0 -0.3"/>
   </joint>
-  <link name="laser">
+  <link name="laser_link">
     <visual>
       <geometry>
@@ -212,5 +212,5 @@
     <axis xyz="0 0 1"/>
     <parent link="body_link"/>
-    <child link="laser"/>
+    <child link="laser_link"/>
     <origin rpy="0 0 0" xyz="0.2 0 0.5"/>
   </joint>

Commit message: updates

File: urdf/sherpa.urdf.xacro (robot description, xacro)
@@ -74,4 +74,187 @@
     </inertial>
   </link>
+  <joint name="camera_joint" type="fixed">
+    <axis xyz="0 0 1"/>
+    <parent link="body_link"/>
+    <child link="camera_link"/>
+    <origin rpy="0 0 0" xyz="0.2 0 -0.3"/>
+  </joint>
+  <link name="laser_link">
+    <visual>
+      <geometry>
+        <box size="0.0762 0.2794 0.0762"/>
+      </geometry>
+      <material name="blue">
+	<color rgba="0.1 0.1 1 1"/>
+      </material>
+    </visual>
+    <collision>
+      <geometry>
+        <box size="0.0762 0.2794 0.0762"/>
+      </geometry>
+    </collision>
+   <inertial>
+      <mass value="0.25"/>
+      <inertia ixx="1.0" iyy="1.0" izz="1.0"
+               ixy="0" ixz="0" iyz="0"/>
+    </inertial>
+  </link>
+  <joint name="laser_joint" type="fixed">
+    <axis xyz="0 0 1"/>
+    <parent link="body_link"/>
+    <child link="laser_link"/>
+    <origin rpy="0 0 0" xyz="0.2 0 0.5"/>
+  </joint>
+  <link name="hitch_front_link">
+    <visual>
+      <geometry>
+        <cylinder length="0.1524" radius="0.01"/>
+      </geometry>
+      <material name="silver">
+	<color rgba="0.75 0.75 0.75 1"/>
+      </material>
+    </visual>
+    <collision>
+      <geometry>
+        <cylinder length="0.1524" radius="0.01"/>
+      </geometry>
+    </collision>
+    <inertial>
+      <mass value="0.1"/>
+      <inertia ixx="1.0" iyy="1.0" izz="1.0"
+               ixy="0" ixz="0" iyz="0"/>
+    </inertial>
+  </link>
+  <joint name="hitch_joint" type="fixed">
+    <axis xyz="0 0 1"/>
+    <parent link="base_link"/>
+    <child link="hitch_front_link"/>
+    <origin rpy="0 0 0" xyz="0.18 0 0.0762"/>
+  </joint>
+  <link name="wheel_front_left">
+    <visual>
+      <geometry>
+        <cylinder length="0.0508" radius="0.0762"/>
+      </geometry>
+      <material name="black">
+        <color rgba="0 0 0 1"/>
+      </material>
+    </visual>
+    <collision>
+      <geometry>
+        <cylinder length="0.0508" radius="0.0762"/>
+      </geometry>
+    </collision>
+    <inertial>
+      <mass value="0.1"/>
+      <inertia ixx="1.0" iyy="1.0" izz="1.0"
+               ixy="0" ixz="0" iyz="0"/>
+    </inertial>
+  </link>
+  <joint name="axis_front_left" type="continuous">
+    <axis xyz="0 0 1"/>
+    <parent link="base_link"/>
+    <child link="wheel_front_left"/>
+    <origin rpy="-1.5708 0 0" xyz="0.165862 0.18034 0"/>
+  </joint>
+ <link name="wheel_front_right">
+    <visual>
+      <geometry>
+        <cylinder length="0.0508" radius="0.0762"/>
+      </geometry>
+      <material name="black"/>
+    </visual>
+    <collision>
+      <geometry>
+        <cylinder length="0.0508" radius="0.0762"/>
+      </geometry>
+    </collision>
+    <inertial>
+      <mass value="0.1"/>
+      <inertia ixx="1.0" iyy="1.0" izz="1.0"
+               ixy="0" ixz="0" iyz="0"/>
+    </inertial>
+  </link>
+  <joint name="axis_front_right" type="continuous">
+    <axis xyz="0 0 1"/>
+    <parent link="base_link"/>
+    <child link="wheel_front_right"/>
+    <origin rpy="-1.5708 0 0" xyz="0.165862 -0.18034 0"/>
+  </joint>
+  <link name="wheel_rear_right">
+    <visual>
+      <geometry>
+        <cylinder length="0.0508" radius="0.0762"/>
+      </geometry>
+      <material name="black"/>
+    </visual>
+    <collision>
+      <geometry>
+        <cylinder length="0.0508" radius="0.0762"/>
+      </geometry>
+    </collision>
+    <inertial>
+      <mass value="0.1"/>
+      <inertia ixx="1.0" iyy="1.0" izz="1.0"
+               ixy="0" ixz="0" iyz="0"/>
+    </inertial>
+  </link>
+  <joint name="axis_rear_right" type="continuous">
+    <axis xyz="0 0 1"/>
+    <parent link="base_link"/>
+    <child link="wheel_rear_right"/>
+    <origin rpy="-1.5708 0 0" xyz="-0.165862 -0.18034 0"/>
+  </joint>
+  <link name="wheel_rear_left">
+    <visual>
+      <geometry>
+        <cylinder length="0.0508" radius="0.0762"/>
+      </geometry>
+      <material name="black"/>
+    </visual>
+    <collision>
+      <geometry>
+        <cylinder length="0.0508" radius="0.0762"/>
+      </geometry>
+    </collision>
+    <inertial>
+      <mass value="0.1"/>
+      <inertia ixx="1.0" iyy="1.0" izz="1.0"
+               ixy="0" ixz="0" iyz="0"/>
+    </inertial>
+    <gazebo reference="wheel_rear_left">
+      <material>Gazebo/Black</material>
+    </gazebo>
+  </link>
+  <joint name="axis_rear_left" type="continuous">
+    <axis xyz="0 0 1"/>
+    <parent link="base_link"/>
+    <child link="wheel_rear_left"/>
+    <origin rpy="-1.5708 0 0" xyz="-0.165862 0.18034 0"/>
+  </joint>
+<!--
+*
+* Gazebo Drivers
+*
+-->
+<gazebo>
+  <plugin name="skid_steer_drive_controller" filename="libgazebo_ros_skid_steer_drive.so">
+    <updateRate>100.0</updateRate>
+    <robotNamespace>/</robotNamespace>
+    <leftFrontJoint>axis_front_left</leftFrontJoint>
+    <rightFrontJoint>axis_front_right</rightFrontJoint>
+    <leftRearJoint>axis_rear_left</leftRearJoint>
+    <rightRearJoint>axis_rear_right</rightRearJoint>
+    <wheelSeparation>0.254</wheelSeparation>
+    <wheelDiameter>0.1524</wheelDiameter>
+    <robotBaseFrame>base_link</robotBaseFrame>
+    <torque>10</torque>
+    <commandTopic>cmd_vel</commandTopic>
+    <broadcastTF>1</broadcastTF>
+  </plugin>
+  <plugin name="joint_state_publisher" filename="libgazebo_ros_joint_state_publisher.so">
+    <jointName>axis_front_left, axis_front_right, axis_rear_left, axis_rear_right</jointName>
+  </plugin>
+</gazebo>
 <!--<xacro:macro name="sim_kinect">
    <gazebo reference="camera_link">
@@ -113,5 +296,5 @@
 </xacro:macro>
 <sim_kinect/>-->
-<gazebo reference="camera_link">
+<!--<gazebo reference="camera_link">
     <sensor type="depth" name="camera">
         <always_on>1</always_on>
@@ -155,5 +338,5 @@
             </plugin>
     </sensor>
-</gazebo>
+</gazebo>-->
 <gazebo reference="laser_link">
     <material>Gazebo/Blue</material>
@@ -183,181 +366,3 @@
     </sensor>
   </gazebo>
-  <joint name="camera_joint" type="fixed">
-    <axis xyz="0 0 1"/>
-    <parent link="body_link"/>
-    <child link="camera_link"/>
-    <origin rpy="0 0 0" xyz="0.2 0 -0.3"/>
-  </joint>
-  <link name="laser_link">
-    <visual>
-      <geometry>
-        <box size="0.0762 0.2794 0.0762"/>
-      </geometry>
-      <material name="blue">
-	<color rgba="0.1 0.1 1 1"/>
-      </material>
-    </visual>
-    <collision>
-      <geometry>
-        <box size="0.0762 0.2794 0.0762"/>
-      </geometry>
-    </collision>
-   <inertial>
-      <mass value="0.25"/>
-      <inertia ixx="1.0" iyy="1.0" izz="1.0"
-               ixy="0" ixz="0" iyz="0"/>
-    </inertial>
-  </link>
-  <joint name="laser_joint" type="fixed">
-    <axis xyz="0 0 1"/>
-    <parent link="body_link"/>
-    <child link="laser_link"/>
-    <origin rpy="0 0 0" xyz="0.2 0 0.5"/>
-  </joint>
-  <link name="hitch_front_link">
-    <visual>
-      <geometry>
-        <cylinder length="0.1524" radius="0.01"/>
-      </geometry>
-      <material name="silver">
-	<color rgba="0.75 0.75 0.75 1"/>
-      </material>
-    </visual>
-    <collision>
-      <geometry>
-        <cylinder length="0.1524" radius="0.01"/>
-      </geometry>
-    </collision>
-    <inertial>
-      <mass value="0.1"/>
-      <inertia ixx="1.0" iyy="1.0" izz="1.0"
-               ixy="0" ixz="0" iyz="0"/>
-    </inertial>
-  </link>
-  <joint name="hitch_joint" type="fixed">
-    <axis xyz="0 0 1"/>
-    <parent link="base_link"/>
-    <child link="hitch_front_link"/>
-    <origin rpy="0 0 0" xyz="0.18 0 0.0762"/>
-  </joint>
-  <link name="wheel_front_left">
-    <visual>
-      <geometry>
-        <cylinder length="0.0508" radius="0.0762"/>
-      </geometry>
-      <material name="black">
-        <color rgba="0 0 0 1"/>
-      </material>
-    </visual>
-    <collision>
-      <geometry>
-        <cylinder length="0.0508" radius="0.0762"/>
-      </geometry>
-    </collision>
-    <inertial>
-      <mass value="0.1"/>
-      <inertia ixx="1.0" iyy="1.0" izz="1.0"
-               ixy="0" ixz="0" iyz="0"/>
-    </inertial>
-  </link>
-  <joint name="axis_front_left" type="continuous">
-    <axis xyz="0 0 1"/>
-    <parent link="base_link"/>
-    <child link="wheel_front_left"/>
-    <origin rpy="-1.5708 0 0" xyz="0.165862 0.18034 0"/>
-  </joint>
- <link name="wheel_front_right">
-    <visual>
-      <geometry>
-        <cylinder length="0.0508" radius="0.0762"/>
-      </geometry>
-      <material name="black"/>
-    </visual>
-    <collision>
-      <geometry>
-        <cylinder length="0.0508" radius="0.0762"/>
-      </geometry>
-    </collision>
-    <inertial>
-      <mass value="0.1"/>
-      <inertia ixx="1.0" iyy="1.0" izz="1.0"
-               ixy="0" ixz="0" iyz="0"/>
-    </inertial>
-  </link>
-  <joint name="axis_front_right" type="continuous">
-    <axis xyz="0 0 1"/>
-    <parent link="base_link"/>
-    <child link="wheel_front_right"/>
-    <origin rpy="-1.5708 0 0" xyz="0.165862 -0.18034 0"/>
-  </joint>
-  <link name="wheel_rear_right">
-    <visual>
-      <geometry>
-        <cylinder length="0.0508" radius="0.0762"/>
-      </geometry>
-      <material name="black"/>
-    </visual>
-    <collision>
-      <geometry>
-        <cylinder length="0.0508" radius="0.0762"/>
-      </geometry>
-    </collision>
-    <inertial>
-      <mass value="0.1"/>
-      <inertia ixx="1.0" iyy="1.0" izz="1.0"
-               ixy="0" ixz="0" iyz="0"/>
-    </inertial>
-  </link>
-  <joint name="axis_rear_right" type="continuous">
-    <axis xyz="0 0 1"/>
-    <parent link="base_link"/>
-    <child link="wheel_rear_right"/>
-    <origin rpy="-1.5708 0 0" xyz="-0.165862 -0.18034 0"/>
-  </joint>
-  <link name="wheel_rear_left">
-    <visual>
-      <geometry>
-        <cylinder length="0.0508" radius="0.0762"/>
-      </geometry>
-      <material name="black"/>
-    </visual>
-    <collision>
-      <geometry>
-        <cylinder length="0.0508" radius="0.0762"/>
-      </geometry>
-    </collision>
-    <inertial>
-      <mass value="0.1"/>
-      <inertia ixx="1.0" iyy="1.0" izz="1.0"
-               ixy="0" ixz="0" iyz="0"/>
-    </inertial>
-    <gazebo reference="wheel_rear_left">
-      <material>Gazebo/Black</material>
-    </gazebo>
-  </link>
-  <joint name="axis_rear_left" type="continuous">
-    <axis xyz="0 0 1"/>
-    <parent link="base_link"/>
-    <child link="wheel_rear_left"/>
-    <origin rpy="-1.5708 0 0" xyz="-0.165862 0.18034 0"/>
-  </joint>
-<gazebo>
-  <plugin name="skid_steer_drive_controller" filename="libgazebo_ros_skid_steer_drive.so">
-    <updateRate>100.0</updateRate>
-    <robotNamespace>/</robotNamespace>
-    <leftFrontJoint>axis_front_left</leftFrontJoint>
-    <rightFrontJoint>axis_front_right</rightFrontJoint>
-    <leftRearJoint>axis_rear_left</leftRearJoint>
-    <rightRearJoint>axis_rear_right</rightRearJoint>
-    <wheelSeparation>0.254</wheelSeparation>
-    <wheelDiameter>0.1524</wheelDiameter>
-    <robotBaseFrame>base_link</robotBaseFrame>
-    <torque>10</torque>
-    <commandTopic>cmd_vel</commandTopic>
-    <broadcastTF>1</broadcastTF>
-  </plugin>
-  <plugin name="joint_state_publisher" filename="libgazebo_ros_joint_state_publisher.so">
-    <jointName>axis_front_left, axis_front_right, axis_rear_left, axis_rear_right</jointName>
-  </plugin>
-</gazebo>
 </robot>

Commit message: Fixed non gpu laser

File: urdf/sherpa.urdf.xacro (robot description, xacro)
@@ -89,9 +89,9 @@
       </material>
     </visual>
-    <collision>
+<!--    <collision>
       <geometry>
         <box size="0.0762 0.2794 0.0762"/>
       </geometry>
-    </collision>
+    </collision> -->
    <inertial>
       <mass value="0.25"/>

Commit message: fixed laser

File: urdf/sherpa.urdf.xacro (robot description, xacro)
@@ -89,9 +89,9 @@
       </material>
     </visual>
-<!--    <collision>
+    <collision>
       <geometry>
         <box size="0.0762 0.2794 0.0762"/>
       </geometry>
-    </collision> -->
+    </collision>
    <inertial>
       <mass value="0.25"/>
@@ -341,5 +341,5 @@
 <gazebo reference="laser_link">
     <material>Gazebo/Blue</material>
-    <sensor type="ray" name="hokuyo">
+    <sensor type="ray" name="head_hokuyo_sensor">
       <pose>0 0 0 0 0 0</pose>
       <visualize>true</visualize>
@@ -350,6 +350,6 @@
             <samples>720</samples>
             <resolution>1</resolution>
-            <min_angle>-1.570796</min_angle>
-            <max_angle>1.570796</max_angle>
+            <min_angle>-2.26889</min_angle>
+            <max_angle>2.26889</max_angle>
           </horizontal>
         </scan>
@@ -360,5 +360,5 @@
         </range>
       </ray>
-      <plugin name="gpu_laser" filename="libgazebo_ros_laser.so">
+      <plugin name="gazebo_ros_head_hokuyo_controller" filename="libgazebo_ros_laser.so">
         <topicName>/scan</topicName>
         <frameName>laser_link</frameName>

Commit message: Turned off colisions for laser

File: urdf/sherpa.urdf.xacro (robot description, xacro)
@@ -89,9 +89,9 @@
       </material>
     </visual>
-    <collision>
+<!--    <collision>
       <geometry>
         <box size="0.0762 0.2794 0.0762"/>
       </geometry>
-    </collision>
+    </collision> -->
    <inertial>
       <mass value="0.25"/>
@@ -104,5 +104,5 @@
     <parent link="body_link"/>
     <child link="laser_link"/>
-    <origin rpy="0 0 0" xyz="0.2 0 0.5"/>
+    <origin rpy="0 0 0" xyz="0.2 0 0.7"/>
   </joint>
   <link name="hitch_front_link">

Commit message: Moved laser to top of robot

File: urdf/sherpa.urdf.xacro (robot description, xacro)
@@ -104,5 +104,5 @@
     <parent link="body_link"/>
     <child link="laser_link"/>
-    <origin rpy="0 0 0" xyz="0.2 0 0.7"/>
+    <origin rpy="0 0 0" xyz="0.2 0 0.55"/>
   </joint>
   <link name="hitch_front_link">
